File: Project/toprevan.kicad_pcb (KiCad board)
At the start: 4 copper layers, 242.9 x 76.2 mm, 122 parts, among them J1 JST SH, J2 Pico EZmate, J3 USB_C_Receptacle_USB2.0, J4 ARGB, SW1 BOOT0, U1 STM32F401CBUx, U3 XC6206PxxxMR, U4 74HC4051, U5 OPA350, U6 74HC4051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

Commit message: review
Routing:
- net GND: track 90.2 -> 92.5 mm, vias 380 -> 386
Other:
- board text added: "JLCJLCJLCJLC"

Commit message: proto ready
Routing:
- net ROW3: vias 11 -> 1
- net ROW2: vias 12 -> 0
- net ROW1: vias 12 -> 0
- net ROW0: vias 12 -> 0
- net COL9: vias 4 -> 0
- net COL8: vias 6 -> 2
- net COL7: vias 4 -> 1
- net COL6: vias 4 -> 0
- net COL5: vias 4 -> 0
- net COL4: vias 4 -> 0
- net COL3: vias 4 -> 1
- net COL2: vias 4 -> 0
- net COL11: vias 6 -> 2
- net COL10: vias 4 -> 0
- net COL1: vias 4 -> 0
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Other:
- outline, holes or cut-outs redrawn
