File: Project/Plates/plate tray split.kicad_pcb (KiCad board)
At the start: 2 copper layers, 243.4 x 76.2 mm, 40 parts

Commit message: publishing changes
Parts:
- removed G***: LOGO, LOGO
- added REF**: Value, cipulot_parts:ecs_plate_cut_1U, F.Cu at (196.8, 88.1)
Other:
- board text removed: "logo by calumwri"
- board text removed: "pcb by Calvin0563"
